File: hardware/Rowing Computer.sch (KiCad schematic (older format))
At the start: 55 parts, among them J1 USB_B_Micro, J2 SWD, J3 Conn_01x02, J4 Micro_SD_Card, J5 Conn_01x31, U1 BQ25895RTW, U2 LP5907MFX-3.3, U3 STM32F042K6Tx, U4 MMA8451QR1, U5 LM2731XMF

Commit message: iteration 2 of board with correct footprint sizes and fixes where solder mask was not applied between pads
Parts:
- L2: footprint Inductor_SMD:L_0603_1608Metric -> Inductor_SMD:L_0805_2012Metric
Changed lines of the file:
@@
 F 0 "L2" H 10950 1315 50  0000 C CNN
 F 1 "33u" H 10950 1224 50  0000 C CNN
-F 2 "Inductor_SMD:L_0603_1608Metric" H 10950 1100 50  0001 C CNN
+F 2 "Inductor_SMD:L_0805_2012Metric" H 10950 1100 50  0001 C CNN
 F 3 "~" H 10950 1100 50  0001 C CNN
 	1    10950 1100
